Commit message: Projekt nr 2 - manipulator - poprawa

File: wizualizacja_manipulatora/urdf/movable.urdf (robot description, URDF)
Before this commit: robot pimpek, 4 links, 3 joints
Joints:
- joint link_2_to_tool: axis (none) -> 1 0 0; limit (none) -> lower=-0.2 upper=0 effort=1000.0 velocity=0.5; type fixed -> prismatic

Commit message: Projekt nr 2 - manipulator - poprawa

File: wizualizacja_manipulatora/urdf/movable.urdf (robot description, URDF)
Before this commit: robot pimpek, 4 links, 3 joints
Joints:
- joint link_2_to_tool: axis 1 0 0 -> 0 0 1; limit lower=-0.2 upper=0 effort=1000.0 velocity=0.5 -> lower=-0.05 upper=0.15 effort=1000.0 velocity=0.5
